File: hardware/backpannel/pcb_files/Ledstrips_PCB.kicad_pcb (KiCad board)
At the start: 2 copper layers, 442 x 467 mm, 51 parts, among them J1 Conn_01x04_Male, J2 Conn_01x02_Female, U1 AMS1117-3.3, U10 WS2812B_strip, U11 WS2812B_strip, U12 WS2812B_strip, U13 WS2812B_strip, U14 WS2812B_strip, U15 WS2812B_strip, U2 ESP-12E, U3 WS2812B_strip, U4 WS2812B_strip, U5 WS2812B_strip, U6 WS2812B_strip, U7 WS2812B_strip, U8 WS2812B_strip, U9 WS2812B_strip

Commit message: Updated PCB and ledschotten
Parts:
- removed the REF** at (83.3, 83.3)
- removed the REF** at (516.7, 350.0)
- removed the REF** at (516.7, 216.6)
- removed the REF** at (516.7, 83.3)
- removed the REF** at (183.3, 183.3)
- removed the REF** at (183.3, 416.6)
- removed the REF** at (416.7, 416.6)
- removed the REF** at (416.7, 183.3)
- removed the REF** at (250.0, 350.0)
- removed the REF** at (350.0, 350.0)
- removed the REF** at (250.0, 250.0)
- removed the REF** at (366.7, 83.3)
- removed the REF** at (349.5, 250.0)
- removed the REF** at (250.0, 83.3)
- removed the REF** at (83.3, 183.3)
- removed the REF** at (83.3, 450.0)
- removed the REF** at (83.3, 316.6)
- removed the REF** at (250.0, 483.3)
- removed the REF** at (350.0, 483.3)
- removed the REF** at (516.7, 483.3)
- removed U10, U11, U12, U13, U14, U15, U3, U4, U5, U6, U7, U8, U9: WS2812B_strip, LED_SMD:ws2812_ledstrip
- added JP1: Reset, Jumper:SolderJumper-2_P1.3mm_Open_RoundedPad1.0x1.5mm, F.Cu at (360.3, 339.2)
- added REF**: MountingHole_3mm, MountingHole:MountingHole_3mm, F.Cu at (500.0, 512.5)
- added REF**: MountingHole_3mm, MountingHole:MountingHole_3mm, F.Cu at (500.0, 712.5)
- added REF**: MountingHole_3mm, MountingHole:MountingHole_3mm, F.Cu at (500.0, 612.5)
- added REF**: MountingHole_3mm, MountingHole:MountingHole_3mm, F.Cu at (600.0, 512.5)
- added REF**: MountingHole_3mm, MountingHole:MountingHole_3mm, F.Cu at (766.7, 612.5)
- added REF**: MountingHole_3mm, MountingHole:MountingHole_3mm, F.Cu at (600.0, 345.8)
- added REF**: MountingHole_3mm, MountingHole:MountingHole_3mm, F.Cu at (333.3, 712.5)
- added REF**: MountingHole_3mm, MountingHole:MountingHole_3mm, F.Cu at (433.3, 512.5)
- added REF**: MountingHole_3mm, MountingHole:MountingHole_3mm, F.Cu at (766.7, 412.5)
- added REF**: MountingHole_3mm, MountingHole:MountingHole_3mm, F.Cu at (500.0, 345.8)
- added REF**: MountingHole_8.4mm_M8, MountingHole:MountingHole_8.4mm_M8, F.Cu at (550.0, 320.7)
- added REF**: MountingHole_8.4mm_M8, MountingHole:MountingHole_8.4mm_M8, F.Cu at (338.7, 320.6)
- added REF**: MountingHole_3mm, MountingHole:MountingHole_3mm, F.Cu at (500.0, 779.1)
- added REF**: MountingHole_3mm, MountingHole:MountingHole_3mm, F.Cu at (433.3, 612.5)
- added REF**: MountingHole_3mm, MountingHole:MountingHole_3mm, F.Cu at (700.0, 712.5)
- added REF**: MountingHole_3mm, MountingHole:MountingHole_3mm, F.Cu at (600.0, 612.5)
- added REF**: MountingHole_3mm, MountingHole:MountingHole_3mm, F.Cu at (333.3, 779.1)
- added REF**: MountingHole_3mm, MountingHole:MountingHole_3mm, F.Cu at (400.0, 345.8)
- added REF**: MountingHole_3mm, MountingHole:MountingHole_3mm, F.Cu at (600.0, 712.5)
- added REF**: MountingHole_3mm, MountingHole:MountingHole_3mm, F.Cu at (766.7, 679.1)
- added REF**: MountingHole_3mm, MountingHole:MountingHole_3mm, F.Cu at (333.3, 512.5)
- added REF**: MountingHole_3mm, MountingHole:MountingHole_3mm, F.Cu at (700.0, 412.5)
- added REF**: MountingHole_3mm, MountingHole:MountingHole_3mm, F.Cu at (400.0, 779.1)
- added REF**: MountingHole_3mm, MountingHole:MountingHole_3mm, F.Cu at (333.3, 612.5)
- added REF**: MountingHole_3mm, MountingHole:MountingHole_3mm, F.Cu at (500.0, 412.5)
- added REF**: MountingHole_3mm, MountingHole:MountingHole_3mm, F.Cu at (766.1, 512.5)
- added REF**: MountingHole_3mm, MountingHole:MountingHole_3mm, F.Cu at (700.0, 345.8)
- added REF**: MountingHole_3mm, MountingHole:MountingHole_3mm, F.Cu at (400.0, 712.5)
- added REF**: MountingHole_3mm, MountingHole:MountingHole_3mm, F.Cu at (766.7, 345.8)
- added REF**: MountingHole_3mm, MountingHole:MountingHole_3mm, F.Cu at (666.7, 612.5)
- added REF**: MountingHole_3mm, MountingHole:MountingHole_3mm, F.Cu at (600.0, 412.5)
- added REF**: MountingHole_3mm, MountingHole:MountingHole_3mm, F.Cu at (766.7, 779.1)
- added REF**: MountingHole_3mm, MountingHole:MountingHole_3mm, F.Cu at (666.7, 512.5)
- added REF**: MountingHole_3mm, MountingHole:MountingHole_3mm, F.Cu at (400.0, 412.5)
- added REF**: MountingHole_3mm, MountingHole:MountingHole_3mm, F.Cu at (600.0, 779.1)
- added REF**: MountingHole_3mm, MountingHole:MountingHole_3mm, F.Cu at (333.3, 345.8)
- added REF**: MountingHole_3mm, MountingHole:MountingHole_3mm, F.Cu at (700.0, 779.1)
- added REF**: MountingHole_3mm, MountingHole:MountingHole_3mm, F.Cu at (333.3, 412.5)
- added REF**: MountingHole_8.4mm_M8, MountingHole:MountingHole_8.4mm_M8, F.Cu at (759.6, 320.7)
- added S1: WS2812_ledstrip, woordklok_footprint:WS2812_ledstrip_30leds_meter, F.Cu at (550.0, 362.4)
- added S10: WS2812_ledstrip, woordklok_footprint:WS2812_ledstrip_30leds_meter, F.Cu at (550.0, 662.4)
- added S11: WS2812_ledstrip, woordklok_footprint:WS2812_ledstrip_30leds_meter, F.Cu at (550.0, 695.8)
- added S12: WS2812_ledstrip, woordklok_footprint:WS2812_ledstrip_30leds_meter, F.Cu at (550.0, 729.1)
- added S13: WS2812_ledstrip, woordklok_footprint:WS2812_ledstrip_30leds_meter, F.Cu at (550.0, 762.4)
- added S2: WS2812_ledstrip, woordklok_footprint:WS2812_ledstrip_30leds_meter, F.Cu at (550.0, 395.8)
- added S3: WS2812_ledstrip, woordklok_footprint:WS2812_ledstrip_30leds_meter, F.Cu at (550.0, 429.1)
- added S4: WS2812_ledstrip, woordklok_footprint:WS2812_ledstrip_30leds_meter, F.Cu at (550.0, 462.4)
- added S5: WS2812_ledstrip, woordklok_footprint:WS2812_ledstrip_30leds_meter, F.Cu at (550.0, 495.8)
- added S6: WS2812_ledstrip, woordklok_footprint:WS2812_ledstrip_30leds_meter, F.Cu at (550.0, 529.1)
- added S7: WS2812_ledstrip, woordklok_footprint:WS2812_ledstrip_30leds_meter, F.Cu at (550.0, 562.4)
- added S8: WS2812_ledstrip, woordklok_footprint:WS2812_ledstrip_30leds_meter, F.Cu at (550.0, 595.8)
- added S9: WS2812_ledstrip, woordklok_footprint:WS2812_ledstrip_30leds_meter, F.Cu at (550.0, 629.1)
- C1, C3: footprint Capacitor_SMD:C_0603_1608Metric_Pad1.08x0.95mm_HandSolder -> Capacitor_SMD:C_0805_2012Metric_Pad1.18x1.45mm_HandSolder
- C2: footprint Capacitor_SMD:CP_Elec_3x5.4 -> Capacitor_SMD:CP_Elec_6.3x5.4
- D1: footprint Diode_SMD:D_0603_1608Metric_Pad1.05x0.95mm_HandSolder -> Diode_SMD:D_0805_2012Metric_Pad1.15x1.40mm_HandSolder
- J1: value Conn_01x04_Male -> Conn_02x03; footprint Connector_PinHeader_2.54mm:PinHeader_1x04_P2.54mm_Vertical -> Connector_PinHeader_2.54mm:PinHeader_2x03_P2.54mm_Vertical
- R1, R10, R3, R4, R5, R6, R7, R8, R9: footprint Resistor_SMD:R_0603_1608Metric_Pad0.98x0.95mm_HandSolder -> Resistor_SMD:R_0805_2012Metric_Pad1.20x1.40mm_HandSolder
- R2: value GL5537 -> LDR; footprint OptoDevice:R_LDR_5.0x4.1mm_P3mm_Vertical -> OptoDevice:R_LDR_5.1x4.3mm_P3.4mm_Vertical
- moved R3 370.1 mm to (373.1, 339.1), turned to 180 degrees
- moved R4 368.8 mm to (369.2, 339.1), turned to 180 degrees
- moved R10 368.7 mm to (363.2, 338.2), turned to 90 degrees
- moved R5 367.4 mm to (366.2, 338.2)
- moved C1 366.7 mm to (404.4, 334.3)
- moved U1 366.6 mm to (397.9, 334.4)
- moved R6 366.0 mm to (373.1, 337.0), turned to 0 degrees
- moved D1 365.9 mm to (397.6, 328.9)
- moved R8 365.5 mm to (376.7, 315.0)
- moved R7 365.5 mm to (374.6, 315.0)
- moved U2 365.3 mm to (369.6, 326.2)
- moved R1 364.7 mm to (369.2, 337.0), turned to 0 degrees
- moved C3 364.6 mm to (380.1, 337.9), turned to -90 degrees
- moved C2 364.4 mm to (388.1, 333.9), turned to 90 degrees
- moved R9 364.4 mm to (378.7, 315.0), turned to -90 degrees
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Connections:
- J1 pad 1: GND -> +3V3
- J1 pad 2: Net-(J1-Pad2) -> /Flash
- J1 pad 3: Net-(J1-Pad3) -> GND
- J1 pad 4: +3V3 -> Net-(R10-Pad2)
- J2 pad 1: GND -> +5V
- J2 pad 2: +5V -> GND
- R10 pad 2: Net-(J1-Pad2) -> Net-(R10-Pad2)
- R5 pad 1: Net-(R5-Pad1) -> /Reset
- R7 pad 2: Net-(R7-Pad2) -> /Flash
- U2 pad 1: Net-(R5-Pad1) -> /Reset
- U2 pad 10: Net-(U2-Pad10) -> unconnected-(U2-Pad10)
- U2 pad 11: Net-(U2-Pad11) -> unconnected-(U2-Pad11)
- U2 pad 12: Net-(U2-Pad12) -> unconnected-(U2-Pad12)
- U2 pad 13: Net-(U2-Pad13) -> unconnected-(U2-Pad13)
- U2 pad 14: Net-(U2-Pad14) -> unconnected-(U2-Pad14)
- U2 pad 18: Net-(R7-Pad2) -> /Flash
- U2 pad 19: Net-(U2-Pad19) -> unconnected-(U2-Pad19)
- U2 pad 20: Net-(U2-Pad20) -> unconnected-(U2-Pad20)
- U2 pad 21: Net-(J1-Pad2) -> Net-(R10-Pad2)
- U2 pad 22: Net-(J1-Pad3) -> Net-(J1-Pad6)
- U2 pad 4: Net-(U2-Pad4) -> unconnected-(U2-Pad4)
- U2 pad 5: Net-(U2-Pad5) -> unconnected-(U2-Pad5)
- U2 pad 6: Net-(U2-Pad6) -> unconnected-(U2-Pad6)
- U2 pad 7: Net-(U2-Pad7) -> unconnected-(U2-Pad7)
- U2 pad 9: Net-(U2-Pad9) -> unconnected-(U2-Pad9)
Routing:
- net +5V: track 64.1 -> 6.85 mm, vias 32 -> 0
- net Net-(U11-Pad2): track 37.6 -> 0.00 mm
- net Net-(U10-Pad2): track 37.6 -> 0.00 mm
- net Net-(U15-Pad2): track 37.6 -> 0.00 mm
- net Net-(U14-Pad2): track 37.6 -> 0.00 mm
- net Net-(U13-Pad2): track 37.6 -> 0.00 mm
- net Net-(U12-Pad2): track 37.6 -> 0.00 mm
- net Net-(U15-Pad4): track 37.6 -> 0.00 mm
- net Net-(U13-Pad4): track 37.6 -> 0.00 mm
- net Net-(U12-Pad4): track 37.6 -> 0.00 mm
- net Net-(U14-Pad4): track 37.6 -> 0.00 mm
- net Net-(U11-Pad4): track 37.6 -> 0.00 mm
- net Net-(U10-Pad4): track 37.6 -> 0.00 mm
- net +3V3: track 42.9 -> 5.68 mm, vias 10 -> 0
- net Net-(JP1-Pad1): track 36.4 -> 2.28 mm
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- added copper zone on F.Cu, net +3V3
- added copper zone on F.Cu, net +5V
- added copper zone on B.Cu, net GND
- removed copper zone on B.Cu, net +3V3
- removed copper zone on B.Cu, net +5V
- removed copper zone on F.Cu, net GND
Other:
- board size 442 x 467 mm -> 440 x 473.5 mm
- net class Default removed

Commit message: update PCB and ngc files for 13x13 clock
Parts:
- JP1: value Reset -> ledstrip
Routing:
- net Net-(S2-Pad4): track 0.00 -> 39.8 mm
- net Net-(S6-Pad4): track 0.00 -> 39.6 mm
- net Net-(S12-Pad4): track 0.00 -> 39.6 mm
- net Net-(S8-Pad4): track 0.00 -> 39.6 mm
- net Net-(S4-Pad4): track 0.00 -> 39.6 mm
- net Net-(S10-Pad4): track 0.00 -> 39.6 mm
- net Net-(S1-Pad4): track 0.00 -> 36.9 mm
- net Net-(S7-Pad4): track 0.00 -> 36.8 mm
- net Net-(S11-Pad4): track 0.00 -> 36.8 mm
- net Net-(S3-Pad4): track 0.00 -> 36.8 mm
- net Net-(S5-Pad4): track 0.00 -> 36.8 mm
- net Net-(S10-Pad2): track 0.00 -> 36.8 mm
- net Net-(JP1-Pad2): track 0.00 -> 36.6 mm
- net +3V3: track 5.68 -> 8.74 mm
- net GND: vias 10 -> 36
Other:
- board size 440 x 473.5 mm -> 441.6 x 473.5 mm

Commit message: Finisched PCB
Parts:
- moved JP1 2.80 mm to (357.5, 339.2)
Connections:
- J2 pad 3: (no net) -> GND
Routing:
- net Net-(J1-Pad4): track 25.0 -> 29.6 mm, vias 0 -> 1
- net GND: track 20.2 -> 23.7 mm, vias 36 -> 39
- net Net-(S1-Pad4): track 36.9 -> 34.1 mm
- net Net-(JP1-Pad1): track 2.28 -> 5.07 mm
- net Net-(S7-Pad4): track 36.8 -> 34.1 mm
- net Net-(S11-Pad4): track 36.8 -> 34.1 mm
- net Net-(S3-Pad4): track 36.8 -> 34.1 mm
- net Net-(S5-Pad4): track 36.8 -> 34.1 mm
- net Net-(S10-Pad2): track 36.8 -> 34.1 mm
- net Net-(JP1-Pad2): track 36.6 -> 34.8 mm
