File: hardware/backpannel/backpannel_pcb_11x11_small/backpannel_pcb_11x11_small.kicad_pcb (KiCad board)
At the start: 2 copper layers, 30 parts, among them J1 Conn_01x02_Female, J2 Conn_02x03, U1 AMS1117-3.3, U2 ESP-12E

Commit message: placement 11x11
Parts:
- S1, S10, S11, S2, S3, S4, S5, S6, S7, S8, S9: footprint woordklok_footprint:WS2812_ledstrip_30leds_meter -> woordklok_footprint:WS2812_ledstrip_60leds_meter
- moved C3 397.3 mm to (-222.8, 2.62)
- moved U1 397.0 mm to (-228.8, 1.60)
- moved D1 388.8 mm to (-220.8, 0.55), turned to -90 degrees
- moved C1 386.5 mm to (-218.6, 2.60), turned to -90 degrees
- moved R6 360.2 mm to (-244.5, -1.52)
- moved J2 357.6 mm to (-237.1, -5.12), turned to 180 degrees
- moved C2 354.4 mm to (-229.9, -7.05)
- moved R4 351.9 mm to (-244.4, 4.28), turned to 0 degrees
- moved R10 350.5 mm to (-277.3, 4.90)
- moved R8 349.9 mm to (-244.5, -7.35), turned to 180 degrees
- moved JP1 349.8 mm to (-280.9, 4.92), turned to 180 degrees
- moved R5 349.7 mm to (-244.5, -3.48), turned to 0 degrees
- moved R1 349.6 mm to (-244.4, 0.40), turned to 0 degrees
- moved R2 349.5 mm to (-197.7, 0.18)
- moved R7 349.4 mm to (-244.5, -5.40)
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Routing:
- net Net-(R1-Pad2): track 0.00 -> 48.6 mm
- net Net-(J2-Pad4): track 0.00 -> 44.5 mm, vias 0 -> 1
- net Net-(J2-Pad6): track 0.00 -> 26.2 mm, vias 0 -> 1
- net /Flash: track 0.00 -> 22.1 mm, vias 0 -> 2
- net /Reset: track 0.00 -> 21.9 mm, vias 0 -> 2
- net Net-(R3-Pad2): track 0.00 -> 19.5 mm, vias 0 -> 2
- net Net-(R6-Pad1): track 0.00 -> 16.3 mm, vias 0 -> 2
- net Net-(R8-Pad2): track 0.00 -> 11.3 mm, vias 0 -> 2
- net GND: track 0.00 -> 7.18 mm, vias 0 -> 8
- net Net-(R9-Pad2): track 0.00 -> 5.53 mm, vias 0 -> 2
- net +3V3: track 0.00 -> 2.96 mm
- added copper zone on F.Cu, net +3V3
- added copper zone on F.Cu, net +5V
- added copper zone on B.Cu, net GND
Other:
- board outline added: 188.7 x 203.5 mm

Commit message: finished hardware for small and big clock
Parts:
- added ?: , , F.Cu at (24.9, -13.9)
- added ?: , , F.Cu at (-75.1, 52.8)
- added ?: , , F.Cu at (25.0, 36.2)
- added ?: , , F.Cu at (-75.0, -30.5)
- added ?: , , F.Cu at (74.8, -30.6)
- added ?: , , F.Cu at (41.7, -63.8)
- added ?: , , F.Cu at (-75.1, 86.2)
- added ?: , , F.Cu at (-41.8, 86.2)
- added ?: , , F.Cu at (75.0, 86.2)
- added ?: , , F.Cu at (74.8, 52.8)
- added ?: , , F.Cu at (41.7, 86.2)
- added ?: , , F.Cu at (-75.0, -63.8)
- added ?: , , F.Cu at (-25.1, 36.1)
- added ?: , , F.Cu at (-41.7, -63.8)
- added ?: , , F.Cu at (-25.0, -13.8)
- added ?: , , F.Cu at (74.8, -63.8)
- moved JP1 248.1 mm to (-50.0, -85.7), turned to 0 degrees
- moved R10 238.8 mm to (-56.4, -85.7), turned to 180 degrees
- moved J1 224.2 mm to (83.9, -88.4)
- moved S3 218.2 mm to (0.00, -5.51)
- moved S5 218.0 mm to (0.00, 61.2)
- moved S4 217.6 mm to (0.00, 27.8)
- moved S2 217.3 mm to (0.00, -38.8)
- moved S10 216.8 mm to (0.00, 44.5)
- moved S1 216.4 mm to (0.00, -72.2)
- moved S9 216.3 mm to (0.00, 11.2)
- moved S8 216.1 mm to (0.00, -22.2)
- moved R2 215.1 mm to (-1.69, -88.3)
- moved S7 215.0 mm to (0.00, -55.5)
- moved C1 214.4 mm to (-24.3, -88.2)
- moved C3 214.4 mm to (-28.4, -88.1)
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Routing:
- net Net-(JP1-Pad2): track 0.00 -> 51.8 mm
- net Net-(S2-Pad2): track 0.00 -> 21.9 mm
- net Net-(S4-Pad2): track 0.00 -> 21.9 mm
- net Net-(S3-Pad2): track 0.00 -> 21.9 mm
- net Net-(S11-Pad4): track 0.00 -> 21.9 mm
- net Net-(S10-Pad4): track 0.00 -> 21.9 mm
- net /Reset: track 21.9 -> 39.9 mm
- net Net-(S1-Pad4): track 0.00 -> 16.7 mm, vias 0 -> 2
- net Net-(S3-Pad4): track 0.00 -> 16.7 mm, vias 0 -> 2
- net Net-(S2-Pad4): track 0.00 -> 16.6 mm, vias 0 -> 2
- net Net-(S11-Pad2): track 0.00 -> 16.6 mm, vias 0 -> 2
- net Net-(S10-Pad2): track 0.00 -> 16.5 mm, vias 0 -> 2
- net Net-(R1-Pad2): track 48.6 -> 59.6 mm, vias 0 -> 1
- net GND: track 7.18 -> 16.4 mm, vias 8 -> 33
- net Net-(R9-Pad2): track 5.53 -> 14.4 mm
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Other:
- board size 188.7 x 203.5 mm -> 190 x 200.6 mm
