File: hardware/backpannel/backpannel_pcb_13x13_big/backpannel_pcb_13x13_big.kicad_pcb (KiCad board)
At the start: 2 copper layers, 441.6 x 473.5 mm, 71 parts, among them J1 Conn_02x03, J2 Conn_01x02_Female, U1 AMS1117-3.3, U2 ESP-12E

Commit message: Added all kinds of nieuw hardware
Parts:
- removed the REF** at (338.7, 320.6)
- removed the REF** at (759.6, 320.7)
- moved REF** 33.4 mm to (766.6, 712.5)
- moved J1 25.3 mm to (394.8, 323.0), turned to 180 degrees
- moved R5 24.1 mm to (387.0, 326.0), turned to 180 degrees
- moved J2 23.9 mm to (415.0, 321.5)
- moved R3 18.4 mm to (391.5, 337.5), turned to -90 degrees
- moved R1 17.8 mm to (387.0, 336.0)
- moved R4 17.8 mm to (387.0, 338.5)
- moved R6 16.0 mm to (387.0, 329.0), turned to 180 degrees
- moved R7 14.7 mm to (387.0, 323.0), turned to 0 degrees
- moved R8 11.4 mm to (387.0, 320.0), turned to 0 degrees
- moved JP1 10.0 mm to (367.5, 339.5)
- moved C3 9.08 mm to (387.0, 332.0), turned to 0 degrees
- moved R9 8.51 mm to (387.0, 317.0), turned to 0 degrees
- moved C2 7.67 mm to (395.0, 330.5)
- moved C1 6.67 mm to (411.0, 333.4)
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Routing:
- net Net-(J1-Pad6): track 3.37 -> 29.2 mm, vias 0 -> 1
- net Net-(R6-Pad1): track 4.02 -> 23.9 mm, vias 0 -> 2
- net Net-(R2-Pad1): track 181.9 -> 162.7 mm
- net /Flash: track 5.76 -> 24.9 mm, vias 0 -> 2
- net Net-(R1-Pad1): track 5.25 -> 23.1 mm
- net Net-(R8-Pad2): track 2.53 -> 18.6 mm, vias 0 -> 2
- net Net-(J1-Pad4): track 29.6 -> 44.6 mm
- net /Reset: track 27.6 -> 40.2 mm, vias 1 -> 2
- net Net-(R9-Pad2): track 2.50 -> 13.2 mm
- net Net-(JP1-Pad2): track 34.8 -> 43.7 mm
- net GND: track 23.7 -> 28.3 mm
- net +3V3: track 8.74 -> 12.0 mm
- net Net-(JP1-Pad1): track 5.07 -> 3.68 mm
Other:
- board size 441.6 x 473.5 mm -> 442 x 473.5 mm
